Commit message: Lidar Package

File: src/ackermann_description/urdf/robot.xacro (robot description, xacro)
@@ -309,5 +309,5 @@
     <!-- LIDAR LINK -->
     <!-- ================================ -->
-    <link name="laser_link">
+    <link name="laser">
         <inertial>
             <origin xyz="0 0 0" rpy="0 0 0" />
@@ -338,5 +338,5 @@
     <joint name="laser_joint" type="fixed">
         <parent link="chassis_link" />
-        <child link="laser_link" />
+        <child link="laser" />
         <!-- LiDAR at front edge + its radius, sitting on top surface -->
         <origin xyz=" 0.1 0.0 ${body_height/2 + lidar_height/2}" rpy="0 0 0" />

Commit message: lidar urdf changes

File: src/ackermann_description/urdf/robot.xacro (robot description, xacro)
@@ -340,5 +340,5 @@
         <child link="laser" />
         <!-- LiDAR at front edge + its radius, sitting on top surface -->
-        <origin xyz=" 0.1 0.0 ${body_height/2 + lidar_height/2}" rpy="0 0 0" />
+        <origin xyz=" 0.15 0.0 ${body_height/2 + lidar_height/2}" rpy="0 0 0" />
     </joint>
 </robot>

Commit message: hardware files updated

File: src/ackermann_description/urdf/robot.xacro (robot description, xacro)
@@ -337,5 +337,5 @@
     </link>
     <joint name="laser_joint" type="fixed">
-        <parent link="chassis_link" />
+        <parent link="base_link" />
         <child link="laser" />
         <!-- LiDAR at front edge + its radius, sitting on top surface -->

Commit message: IMU bno055 package added

File: src/ackermann_description/urdf/robot.xacro (robot description, xacro)
@@ -5,7 +5,7 @@
     <!-- ================================ -->
     <xacro:property name="body_mass" value="1.58" />
-    <xacro:property name="body_length" value="0.475" />
+    <xacro:property name="body_length" value="0.460" />
     <xacro:property name="body_width" value="0.21" />
-    <xacro:property name="body_height" value="0.160" />
+    <xacro:property name="body_height" value="0.110" />
     <xacro:property name="wheelbase" value="0.285" />
     <xacro:property name="track_width" value="0.280" />
@@ -337,8 +337,34 @@
     </link>
     <joint name="laser_joint" type="fixed">
-        <parent link="base_link" />
+        <parent link="chassis_link" />
         <child link="laser" />
         <!-- LiDAR at front edge + its radius, sitting on top surface -->
         <origin xyz=" 0.15 0.0 ${body_height/2 + lidar_height/2}" rpy="0 0 0" />
     </joint>
+    <!-- ================================ -->
+    <!-- IMU LINK -->
+    <!-- ================================ -->
+    <link name="imu_link">
+        <visual>
+            <origin xyz="0 0 0" rpy="0 0 0" />
+            <geometry>
+                <box size ="0.03 0.03 0.01" />
+            </geometry>
+            <material name="imu_blue">
+                <color rgba="0.1 0.1 0.8 1.0" />
+            </material>
+        </visual>
+        <collision>
+            <origin xyz="0 0 0" rpy="0 0 0" />
+            <geometry>
+                <box size ="0.03 0.03 0.01" />
+            </geometry>
+        </collision>
+    </link>
+    <joint name="imu_joint" type="fixed">
+        <parent link="chassis_link" />
+        <child link="imu_link" />
+        <!-- IMU fixed at center of chassis link-->
+        <origin xyz=" 0.02 0 0.0175" rpy="0 0 0" />
+    </joint>
 </robot>

Commit message: robot localization using EKF

File: src/ackermann_description/urdf/robot.xacro (robot description, xacro)
@@ -366,5 +366,5 @@
         <child link="imu_link" />
         <!-- IMU fixed at center of chassis link-->
-        <origin xyz=" 0.02 0 0.0175" rpy="0 0 0" />
+        <origin xyz=" 0.02 0 ${(body_height/2)+0.0175}" rpy="0 0 0" />
     </joint>
 </robot>

Commit message: Nav tuning

File: src/ackermann_description/urdf/robot.xacro (robot description, xacro)
@@ -15,5 +15,5 @@
     <xacro:property name="steering_mass" value="0.02" />
     <!-- max steering = 45 deg -->
-    <xacro:property name="max_steering_angle" value="${pi/4}" />
+    <xacro:property name="max_steering_angle" value="${7*pi/36}" />
     <xacro:property name="lidar_radius" value="0.035" />
     <xacro:property name="lidar_height" value="0.055" />
